File: molex8/molex8.kicad_pcb (KiCad board)
At the start: 2 copper layers, 42 x 42 mm, 7 parts, among them J1 2xMVE252-5-V, J2 TME 39281083 MOLEX, J3 2xMVE252-5-V

Commit message: molex8: add wire names.
Connections:
- net Net-(J1-Pin_1) renamed /1
- net Net-(J1-Pin_2) renamed /2
- net Net-(J1-Pin_3) renamed /3
- net Net-(J1-Pin_4) renamed /4
- net Net-(J2-Pin_5) renamed /5
- net Net-(J2-Pin_6) renamed /6
- net Net-(J2-Pin_7) renamed /7
- net Net-(J2-Pin_8) renamed /8
